Commit message: Fix launch file with new frame parameters. Update zed urdf

File: urdf/zed.urdf (robot description, URDF)
Before this commit: robot zed_camera, 3 links, 2 joints
Links:
- removed link ZED_center
- removed link ZED_left_camera
- removed link ZED_right_camera
- added link zed_center; visual mesh filename=package://zed_wrapper/urdf/ZED.stl
- added link zed_depth_frame
- added link zed_left_camera; visual cylinder length=.031 radius=0.007
- added link zed_right_camera; visual cylinder length=.031 radius=0.007
Joints:
- removed joint ZED_center_joint
- removed joint ZED_right_camera_joint
- added joint zed_depth_camera_joint: type fixed, parent zed_left_camera, child zed_depth_frame, origin xyz=0 0 0 rpy=-1.5707963267948966 0 -1.5707963267948966
- added joint zed_left_camera_joint: type fixed, parent zed_center, child zed_left_camera, origin xyz=0 0.06 0 rpy=0 0 0
- added joint zed_right_camera_joint: type fixed, parent zed_center, child zed_right_camera, origin xyz=0 -0.06 0 rpy=0 0 0

Commit message: Fix depth cloud warning and improve launch files

File: urdf/zed.urdf (robot description, URDF)
Before this commit: robot zed_camera, 4 links, 3 joints
Links:
- removed link zed_depth_frame
- added link zed_depth_camera
Joints:
- joint zed_depth_camera_joint: child zed_depth_frame -> zed_depth_camera

Commit message: Reorganized ZED TF Tree according to ROS conventions

File: urdf/zed.urdf (robot description, URDF)
Before this commit: robot zed_camera, 4 links, 3 joints
Links:
- removed link zed_depth_camera
- removed link zed_left_camera
- removed link zed_right_camera
- added link zed_left_camera_frame
- added link zed_left_camera_optical_frame
- added link zed_right_camera_frame
- added link zed_right_camera_optical_frame
Joints:
- removed joint zed_depth_camera_joint
- added joint zed_left_camera_optical_joint: type fixed, parent zed_left_camera_frame, child zed_left_camera_optical_frame, origin xyz=0 0 0 rpy=-1.57079632679 0.0 -1.57079632679
- added joint zed_right_camera_optical_joint: type fixed, parent zed_right_camera_frame, child zed_right_camera_optical_frame, origin xyz=0 0 0 rpy=-1.57079632679 0.0 -1.57079632679
- joint zed_left_camera_joint: child zed_left_camera -> zed_left_camera_frame
- joint zed_right_camera_joint: child zed_right_camera -> zed_right_camera_frame

File: urdf/zedm.urdf (robot description, URDF)
Before this commit: robot zedm_camera, 5 links, 4 joints
Links:
- removed link zed_depth_camera
- removed link zed_left_camera
- removed link zed_right_camera
- added link zed_left_camera_frame
- added link zed_left_camera_optical_frame
- added link zed_right_camera_frame
- added link zed_right_camera_optical_frame
- link zed_center: geometry visual mesh filename=package://zed_wrapper/urdf/ZED.stl
Joints:
- removed joint zed_depth_camera_joint
- added joint zed_left_camera_optical_joint: type fixed, parent zed_left_camera_frame, child zed_left_camera_optical_frame, origin xyz=0 0 0 rpy=-1.57079632679 0.0 -1.57079632679
- added joint zed_right_camera_optical_joint: type fixed, parent zed_right_camera_frame, child zed_right_camera_optical_frame, origin xyz=0 0 0 rpy=-1.57079632679 0.0 -1.57079632679
- joint imu_link_joint: parent zed_center -> zed_left_camera_frame
- joint zed_left_camera_joint: child zed_left_camera -> zed_left_camera_frame
- joint zed_right_camera_joint: child zed_right_camera -> zed_right_camera_frame

Commit message: Exposed enable_pose_smoothing and enable_spatial_memory params for tracking  * added a new enable_tracking function  * renamed zed_center to zed_camera_center  * started to work on IMU frame TF publishing

File: urdf/zed.urdf (robot description, URDF)
Before this commit: robot zed_camera, 5 links, 4 joints
Links:
- removed link zed_center
- added link zed_camera_center; visual mesh filename=package://zed_wrapper/urdf/ZED.stl
Joints:
- joint zed_left_camera_joint: parent zed_center -> zed_camera_center
- joint zed_right_camera_joint: parent zed_center -> zed_camera_center

File: urdf/zedm.urdf (robot description, URDF)
Before this commit: robot zedm_camera, 6 links, 5 joints
Links:
- removed link zed_center
- added link zed_camera_center; visual mesh filename=package://zed_wrapper/urdf/ZED.stl
Joints:
- joint imu_link_joint: parent zed_left_camera_frame -> zed_camera_center; type fixed -> floating
- joint zed_left_camera_joint: parent zed_center -> zed_camera_center
- joint zed_right_camera_joint: parent zed_center -> zed_camera_center

Commit message: Added "base_link" frame to help the integration with robots

File: urdf/zed.urdf (robot description, URDF)
Before this commit: robot zed_camera, 5 links, 4 joints
Links:
- added link base_link
- link zed_camera_center: geometry visual mesh filename=package://zed_wrapper/urdf/models/ZED.stl
Joints:
- added joint zed_camera_center_joint: type fixed, parent base_link, child zed_camera_center, origin xyz=0 0.0 0 rpy=0 0 0

File: urdf/zedm.urdf (robot description, URDF)
Before this commit: robot zedm_camera, 6 links, 5 joints
Links:
- added link base_link
- link zed_camera_center: geometry visual mesh filename=package://zed_wrapper/urdf/models/ZEDM.stl
Joints:
- added joint zed_camera_center_joint: type fixed, parent base_link, child zed_camera_center, origin xyz=0 0.0 0 rpy=0 0 0

Commit message: Fixed the problem of the "fliyng robot" with Terrain Mapping initializing the "odom" with the first pose obtained when tracking exits from "SEARCHING"

File: urdf/zed.urdf (robot description, URDF)
Before this commit: robot zed_camera, 6 links, 5 joints
Joints:
- joint zed_camera_center_joint: origin xyz=0 0.0 0 rpy=0 0 0 -> xyz=0 0 0 rpy=0 0 0

File: urdf/zedm.urdf (robot description, URDF)
Before this commit: robot zedm_camera, 7 links, 6 joints
Joints:
- joint zed_camera_center_joint: origin xyz=0 0.0 0 rpy=0 0 0 -> xyz=0 0 0 rpy=0 0 0
