Commit message: Corrected issue with IMU reference frame  * modified coordinate_system to COORDINATE_SYSTEM_RIGHT_HANDED_Z_UP  * correct the coordinate system to COORDINATE_SYSTEM_RIGHT_HANDED_Z_UP_X_FWD as soon as it will be available in SDK  * added a frame_id for IMU  * added a link for IMU

File: urdf/zedm.urdf (robot description, URDF)
Before this commit: robot zedm_camera, 4 links, 3 joints
Links:
- added link imu_link
Joints:
- added joint imu_link_joint: type fixed, parent zed_center, child imu_link, origin xyz=0 0 0 rpy=0 0 0

Commit message: v2.5 merge (#236)
* Updated wrapper compatibility with ZED SDK 2.5.

* Updated "package.xml" to "Format 2"

* Refactored wrapper code for clarity

* Updated publishing rules to stream Odometry when subscribing to point cloud topics

* Added launch example to run wrapper nodelet in a standalone nodelet manager

* Added a publisher for internal IMU data

* Added a publisher for disparity image

* Added parameters for Pose Smoothing and Spatial Memory.

* Added initial tracking position parameter

* Added dynamic image/measures resolution setting to allow compute and bandwidth optimizations

* Fixed minor bugs

File: urdf/zedm.urdf (robot description, URDF)
Before this commit: robot zedm_camera, 4 links, 3 joints
Links:
- removed link zed_center
- removed link zed_depth_camera
- removed link zed_left_camera
- removed link zed_right_camera
- added link imu_link
- added link zed_camera_center; visual mesh filename=package://zed_wrapper/urdf/ZED.stl
- added link zed_left_camera_frame
- added link zed_left_camera_optical_frame
- added link zed_right_camera_frame
- added link zed_right_camera_optical_frame
Joints:
- removed joint zed_depth_camera_joint
- added joint imu_link_joint: type floating, parent zed_camera_center, child imu_link, origin xyz=0 0 0 rpy=0 0 0
- added joint zed_left_camera_optical_joint: type fixed, parent zed_left_camera_frame, child zed_left_camera_optical_frame, origin xyz=0 0 0 rpy=-1.57079632679 0.0 -1.57079632679
- added joint zed_right_camera_optical_joint: type fixed, parent zed_right_camera_frame, child zed_right_camera_optical_frame, origin xyz=0 0 0 rpy=-1.57079632679 0.0 -1.57079632679
- joint zed_left_camera_joint: child zed_left_camera -> zed_left_camera_frame; parent zed_center -> zed_camera_center
- joint zed_right_camera_joint: child zed_right_camera -> zed_right_camera_frame; parent zed_center -> zed_camera_center

Commit message: Manual merge with the "devel_tf" branch to add "base_link" between "zed_camera_center" and "odom" frames for compatibility with external stacks

File: urdf/zedm.urdf (robot description, URDF)
Before this commit: robot zedm_camera, 6 links, 5 joints
Links:
- added link base_link
- link zed_camera_center: geometry visual mesh filename=package://zed_wrapper/urdf/models/ZEDM.stl
Joints:
- added joint zed_camera_center_joint: type fixed, parent base_link, child zed_camera_center, origin xyz=0 0.0 0 rpy=0 0 0

Commit message: Fix zedm model in zedm.urdf

File: urdf/zedm.urdf (robot description, URDF)
Before this commit: robot zedm_camera, 6 links, 5 joints
Links:
- link zed_camera_center: geometry visual mesh filename=package://zed_wrapper/urdf/ZEDM.stl
