Commit message: Moved camera 3D models to their own folder Fixed camera_model param Fixed Dynamic Params

File: zed_wrapper/urdf/zed.urdf (robot description, URDF)
Before this commit: robot zed_camera, 5 links, 4 joints
Links:
- link zed_camera_center: geometry visual mesh filename=package://zed_wrapper/urdf/models/ZED.stl

File: zed_wrapper/urdf/zedm.urdf (robot description, URDF)
Before this commit: robot zedm_camera, 6 links, 5 joints
Links:
- link zed_camera_center: geometry visual mesh filename=package://zed_wrapper/urdf/models/ZEDM.stl

Commit message: Added base_link

File: zed_wrapper/urdf/zed.urdf (robot description, URDF)
Before this commit: robot zed_camera, 5 links, 4 joints
Links:
- added link base_link
Joints:
- added joint zed_camera_center_joint: type fixed, parent base_link, child zed_camera_center, origin xyz=0 0 0 rpy=0 0 0

File: zed_wrapper/urdf/zedm.urdf (robot description, URDF)
Before this commit: robot zedm_camera, 6 links, 5 joints
Links:
- added link base_link
Joints:
- added joint zed_camera_center_joint: type fixed, parent base_link, child zed_camera_center, origin xyz=0 0 0 rpy=0 0 0
