Commit message: Removed the "imu_link" from URDF since it is dinamically published by the node

File: zed_wrapper/urdf/zedm.urdf (robot description, URDF)
Before this commit: robot zedm_camera, 7 links, 6 joints
Links:
- removed link imu_link
Joints:
- removed joint imu_link_joint

Commit message: Started to integrate the new code about odometry twist... not yet working

File: zed_wrapper/urdf/zedm.urdf (robot description, URDF)
Before this commit: robot zedm_camera, 6 links, 5 joints
Joints:
- joint zed_camera_center_joint: origin xyz=0 0 0 rpy=0 0 0 -> xyz=0 0 0.6 rpy=0 0 0

Commit message: minor changes

File: zed_wrapper/urdf/zedm.urdf (robot description, URDF)
Before this commit: robot zedm_camera, 6 links, 5 joints
Joints:
- joint zed_camera_center_joint: origin xyz=0 0 0.6 rpy=0 0 0 -> xyz=0 0 0.0 rpy=0 0 0

Commit message: Merged Diagnostic from "master" branch

File: zed_wrapper/urdf/zedm.urdf (robot description, URDF)
Before this commit: robot zedm_camera, 6 links, 5 joints
Joints:
- joint zed_camera_center_joint: origin xyz=0 0 0.0 rpy=0 0 0 -> xyz=0 0 0.6 rpy=0 0 0

Commit message: Merge from master almost complete. To be checked

File: zed_wrapper/urdf/zedm.urdf (robot description, URDF)
Before this commit: robot zedm_camera, 6 links, 5 joints
Joints:
- joint zed_camera_center_joint: origin xyz=0 0 0.6 rpy=0 0 0 -> xyz=0 0 0.61 rpy=0 0 0

Commit message: Fixed IMU reference frame

File: zed_wrapper/urdf/zedm.urdf (robot description, URDF)
Before this commit: robot zedm_camera, 7 links, 6 joints
Links:
- removed link imu_link
- added link zed_imu_link
Joints:
- joint imu_link_joint: child imu_link -> zed_imu_link

Commit message: Change Elaboration time calculation

File: zed_wrapper/urdf/zedm.urdf (robot description, URDF)
Before this commit: robot zedm_camera, 7 links, 6 joints
Links:
- removed link zed_imu_link
Joints:
- removed joint imu_link_joint
