Commit message: Fix urdf sensors zed2

File: zed_wrapper/urdf/zed.urdf.xacro (robot description, xacro)
@@ -71,4 +71,31 @@
         </joint>
         <link name="${camera_name}_right_camera_optical_frame"/>
+<!-- ZED2 Sensors -->
+        <xacro:if value="${camera_model == 'zed2'}">
+            <joint name="${camera_name}_mag_joint" type="fixed">
+                <parent link="${camera_name}_camera_center"/>
+                <child link="${camera_name}_mag_link"/>
+                <origin xyz="0 0 0" rpy="0 0 0" />
+            </joint>
+            <link name="${camera_name}_mag_link" />
+            <joint name="${camera_name}_baro_joint" type="fixed">
+                <parent link="${camera_name}_camera_center"/>
+                <child link="${camera_name}_baro_link"/>
+                <origin xyz="0 0 0" rpy="0 0 0" />
+            </joint>
+            <link name="${camera_name}_baro_link" />
+            <joint name="${camera_name}_temp_left_joint" type="fixed">
+                <parent link="${camera_name}_left_camera_frame"/>
+                <child link="${camera_name}_temp_left_link"/>
+                <origin xyz="0 0 0" rpy="0 0 0" />
+            </joint>
+            <link name="${camera_name}_temp_left_link" />
+            <joint name="${camera_name}_temp_right_joint" type="fixed">
+                <parent link="${camera_name}_right_camera_frame"/>
+                <child link="${camera_name}_temp_right_link"/>
+                <origin xyz="0 0 0" rpy="0 0 0" />
+            </joint>
+            <link name="${camera_name}_temp_right_link" />
+        </xacro:if>
     </xacro:macro>
 </robot>
