Commit message: Improve URDF link positions

File: zed_wrapper/urdf/zed_macro.urdf.xacro (robot description, xacro)
@@ -29,16 +29,28 @@
       <xacro:property name="baseline" value="0.12" />
       <xacro:property name="height" value="0.033" />
+      <xacro:property name="bottom_slope" value="0.05" />
+      <xacro:property name="screw_offset_x" value="0.0" />
+      <xacro:property name="optical_offset_x" value="-0.01" />
     </xacro:if>
     <xacro:if value="${model == 'zedm'}">
       <xacro:property name="baseline" value="0.06" />
       <xacro:property name="height" value="0.0265" />
+      <xacro:property name="bottom_slope" value="0.0" />
+      <xacro:property name="screw_offset_x" value="0.0" />
+      <xacro:property name="optical_offset_x" value="0.0" />
     </xacro:if>
     <xacro:if value="${model == 'zed2'}">
       <xacro:property name="baseline" value="0.12" />
       <xacro:property name="height" value="0.033" />
+      <xacro:property name="bottom_slope" value="0.05" />
+      <xacro:property name="screw_offset_x" value="0.0" />
+      <xacro:property name="optical_offset_x" value="-0.01" />
     </xacro:if>
     <xacro:if value="${model == 'zed2i'}">
       <xacro:property name="baseline" value="0.12" />
       <xacro:property name="height" value="0.033" />
+      <xacro:property name="bottom_slope" value="0.0" />
+      <xacro:property name="screw_offset_x" value="-0.01" />
+      <xacro:property name="optical_offset_x" value="-0.01" />
     </xacro:if>
     <!-- Camera mounting point (the threaded screw hole in the bottom) -->
@@ -52,5 +64,5 @@
     <link name="${name}_camera_center">
       <visual>
-        <origin xyz="0 0 0" rpy="0 0 0"/>
+        <origin xyz="${screw_offset_x} 0 0" rpy="0 0 0"/>
         <geometry>
           <mesh filename="package://zed_interfaces/meshes/${model}.stl" />
@@ -67,5 +79,5 @@
       <parent link="${name}_base_link"/>
       <child link="${name}_camera_center"/>
-      <origin xyz="0 0 ${height/2}" rpy="0 0 0" />
+      <origin xyz="0 0 ${height/2}" rpy="0 ${bottom_slope} 0" />
     </joint>
     <!-- Left Camera -->
@@ -78,5 +90,5 @@
     <link name="${name}_left_camera_optical_frame"/>
     <joint name="${name}_left_camera_optical_joint" type="fixed">
-      <origin xyz="0 0 0" rpy="-${M_PI/2} 0.0 -${M_PI/2}"/>
+      <origin xyz="${optical_offset_x} 0 0" rpy="-${M_PI/2} 0.0 -${M_PI/2}"/>
       <parent link="${name}_left_camera_frame"/>
       <child link="${name}_left_camera_optical_frame"/>
@@ -91,5 +103,5 @@
     <link name="${name}_right_camera_optical_frame"/>
     <joint name="${name}_right_camera_optical_joint" type="fixed">
-      <origin xyz="0 0 0" rpy="-${M_PI/2} 0.0 -${M_PI/2}"/>
+      <origin xyz="${optical_offset_x} 0 0" rpy="-${M_PI/2} 0.0 -${M_PI/2}"/>
       <parent link="${name}_right_camera_frame"/>
       <child link="${name}_right_camera_optical_frame"/>

Commit message: Fix wrong ZED, ZED2, and ZED2i height value

File: zed_wrapper/urdf/zed_macro.urdf.xacro (robot description, xacro)
@@ -28,5 +28,5 @@
     <xacro:if value="${model == 'zed'}">
       <xacro:property name="baseline" value="0.12" />
-      <xacro:property name="height" value="0.033" />
+      <xacro:property name="height" value="0.03" />
       <xacro:property name="bottom_slope" value="0.05" />
       <xacro:property name="screw_offset_x" value="0.0" />
@@ -42,5 +42,5 @@
     <xacro:if value="${model == 'zed2'}">
       <xacro:property name="baseline" value="0.12" />
-      <xacro:property name="height" value="0.033" />
+      <xacro:property name="height" value="0.03" />
       <xacro:property name="bottom_slope" value="0.05" />
       <xacro:property name="screw_offset_x" value="0.0" />
@@ -49,5 +49,5 @@
     <xacro:if value="${model == 'zed2i'}">
       <xacro:property name="baseline" value="0.12" />
-      <xacro:property name="height" value="0.033" />
+      <xacro:property name="height" value="0.03" />
       <xacro:property name="bottom_slope" value="0.0" />
       <xacro:property name="screw_offset_x" value="-0.01" />
