Commit message: Add Camera position and orientation in launch files Rename `spatial_memory` to `area_memory` Remove zed_multi_cam.launch and zed_multi_gpu.launch Rename `point_cloud/fused_cloud_registered` to `mapping/fused_cloud`

File: zed_wrapper/urdf/zed_descr.urdf.xacro (robot description, xacro)
@@ -21,10 +21,10 @@
     <xacro:arg name="camera_name"   default="zed" />
     <xacro:arg name="camera_model"  default="zed" />
-    <xacro:arg name="pos_x"             default="0.0" />
-    <xacro:arg name="pos_y"             default="0.0" />
-    <xacro:arg name="pos_z"             default="0.0" />
-    <xacro:arg name="roll"          default="0.0" />
-    <xacro:arg name="pitch"         default="0.0" />
-    <xacro:arg name="yaw"           default="0.0" />
+    <xacro:arg name="cam_pos_x"     default="0.0" />
+    <xacro:arg name="cam_pos_y"     default="0.0" />
+    <xacro:arg name="cam_pos_z"     default="0.0" />
+    <xacro:arg name="cam_roll"      default="0.0" />
+    <xacro:arg name="cam_pitch"     default="0.0" />
+    <xacro:arg name="cam_yaw"       default="0.0" />
     <!-- Properties -->
     <xacro:property name="M_PI"     value="3.1415926535897931" />
@@ -45,5 +45,5 @@
         <parent link="base_link"/>
         <child link="$(arg camera_name)_camera_center"/>
-        <origin xyz="$(arg pos_x) $(arg pos_y) $(arg pos_z)" rpy="$(arg roll) $(arg pitch) $(arg yaw)" />
+        <origin xyz="$(arg cam_pos_x) $(arg cam_pos_y) $(arg cam_pos_z)" rpy="$(arg cam_roll) $(arg cam_pitch) $(arg cam_yaw)" />
     </joint>
     <link name="$(arg camera_name)_camera_center">

Commit message: ZED2 sensors frames

File: zed_wrapper/urdf/zed_descr.urdf.xacro (robot description, xacro)
@@ -82,3 +82,30 @@
     </joint>
     <link name="$(arg camera_name)_right_camera_optical_frame"/>
+<!-- ZED2 Sensors -->
+    <xacro:if value="${model == 'zed2'}">
+        <joint name="$(arg camera_name)_mag_joint" type="fixed">
+            <parent link="$(arg camera_name)_camera_center"/>
+            <child link="$(arg camera_name)_mag_link"/>
+            <origin xyz="0 0 0" rpy="0 0 0" />
+        </joint>
+        <link name="$(arg camera_name)_mag_link" />
+        <joint name="$(arg camera_name)_baro_joint" type="fixed">
+            <parent link="$(arg camera_name)_camera_center"/>
+            <child link="$(arg camera_name)_baro_link"/>
+            <origin xyz="0 0 0" rpy="0 0 0" />
+        </joint>
+        <link name="$(arg camera_name)_baro_link" />
+        <joint name="$(arg camera_name)_temp_left_joint" type="fixed">
+            <parent link="$(arg camera_name)_left_camera_frame"/>
+            <child link="$(arg camera_name)_temp_left_link"/>
+            <origin xyz="0 0 0" rpy="0 0 0" />
+        </joint>
+        <link name="$(arg camera_name)_temp_left_link" />
+        <joint name="$(arg camera_name)_temp_right_joint" type="fixed">
+            <parent link="$(arg camera_name)_right_camera_frame"/>
+            <child link="$(arg camera_name)_temp_right_link"/>
+            <origin xyz="0 0 0" rpy="0 0 0" />
+        </joint>
+        <link name="$(arg camera_name)_temp_right_link" />
+    </xacro:if>
 </robot>

Commit message: Now you can include zed.urdf.xacro in another xacro

File: zed_wrapper/urdf/zed_descr.urdf.xacro (robot description, xacro)
@@ -17,5 +17,5 @@
 <robot name="stereolabs_camera" xmlns:xacro="http://ros.org/wiki/xacro">
 <!-- Includes -->
-    <xacro:include filename="$(find zed_wrapper)/urdf/include/materials.urdf.xacro" />
+    <xacro:include filename="$(find zed_wrapper)/urdf/zed.urdf.xacro" />
     <!-- Arguments -->
     <xacro:arg name="camera_name"   default="zed" />
@@ -27,58 +27,9 @@
     <xacro:arg name="cam_pitch"     default="0.0" />
     <xacro:arg name="cam_yaw"       default="0.0" />
-    <!-- Properties -->
-    <xacro:property name="M_PI"     value="3.1415926535897931" />
-    <xacro:property name="model"    value="$(arg camera_model)" />
-    <xacro:if value="${model == 'zed'}">
-        <xacro:property name="baseline" value="0.12" />
-    </xacro:if>
-    <xacro:if value="${model == 'zedm'}">
-        <xacro:property name="baseline" value="0.06" />
-    </xacro:if>
-    <xacro:if value="${model == 'zed2'}">
-        <xacro:property name="baseline" value="0.12" />
-    </xacro:if>
 <!-- base_link -->
     <link name="base_link" />
-<!-- Camera Center -->
-    <joint name="$(arg camera_name)_camera_center_joint" type="fixed">
-        <parent link="base_link"/>
-        <child link="$(arg camera_name)_camera_center"/>
+<!-- zed_macro -->
+    <xacro:zed camera_model="$(arg camera_model)" camera_name="$(arg camera_name)" parent="base_link">
         <origin xyz="$(arg cam_pos_x) $(arg cam_pos_y) $(arg cam_pos_z)" rpy="$(arg cam_roll) $(arg cam_pitch) $(arg cam_yaw)" />
-    </joint>
-    <link name="$(arg camera_name)_camera_center">
-        <visual>
-            <origin xyz="0 0 0" rpy="0 0 0"/>
-            <geometry>
-                <mesh filename="package://zed_wrapper/urdf/models/${model}.stl" />
-            </geometry>
-            <material name="${model}_mat" />
-        </visual>
-    </link>
-<!-- Left Camera -->
-    <joint name="$(arg camera_name)_left_camera_joint" type="fixed">
-        <parent link="$(arg camera_name)_camera_center"/>
-        <child link="$(arg camera_name)_left_camera_frame"/>
-        <origin xyz="0 ${baseline/2} 0" rpy="0 0 0" />
-    </joint>
-    <link name="$(arg camera_name)_left_camera_frame" />
-    <joint name="$(arg camera_name)_left_camera_optical_joint" type="fixed">
-        <origin xyz="0 0 0" rpy="-${M_PI/2} 0.0 -${M_PI/2}"/>
-        <parent link="$(arg camera_name)_left_camera_frame"/>
-        <child link="$(arg camera_name)_left_camera_optical_frame"/>
-    </joint>
-    <link name="$(arg camera_name)_left_camera_optical_frame"/>
-<!-- Right Camera -->
-    <joint name="$(arg camera_name)_right_camera_joint" type="fixed">
-        <parent link="$(arg camera_name)_camera_center"/>
-        <child link="$(arg camera_name)_right_camera_frame"/>
-        <origin xyz="0 -${baseline/2} 0" rpy="0 0 0" />
-    </joint>
-    <link name="$(arg camera_name)_right_camera_frame" />
-    <joint name="$(arg camera_name)_right_camera_optical_joint" type="fixed">
-        <origin xyz="0 0 0" rpy="-${M_PI/2} 0.0 -${M_PI/2}"/>
-        <parent link="$(arg camera_name)_right_camera_frame"/>
-        <child link="$(arg camera_name)_right_camera_optical_frame"/>
-    </joint>
-    <link name="$(arg camera_name)_right_camera_optical_frame"/>
+    </xacro:zed>
 </robot>

Commit message: Propagate `base_frame` parameter in the Xacro description

File: zed_wrapper/urdf/zed_descr.urdf.xacro (robot description, xacro)
@@ -21,4 +21,5 @@
     <xacro:arg name="camera_name"   default="zed" />
     <xacro:arg name="camera_model"  default="zed" />
+    <xacro:arg name="base_frame"    default="base_link" />
     <xacro:arg name="cam_pos_x"     default="0.0" />
     <xacro:arg name="cam_pos_y"     default="0.0" />
@@ -40,8 +41,8 @@
     </xacro:if>
 <!-- base_link -->
-    <link name="base_link" />
+    <link name="$(arg base_frame)" />
 <!-- Camera Center -->
     <joint name="$(arg camera_name)_camera_center_joint" type="fixed">
-        <parent link="base_link"/>
+        <parent link="$(arg base_frame)"/>
         <child link="$(arg camera_name)_camera_center"/>
         <origin xyz="$(arg cam_pos_x) $(arg cam_pos_y) $(arg cam_pos_z)" rpy="$(arg cam_roll) $(arg cam_pitch) $(arg cam_yaw)" />

Commit message: V3.1 (#528)
* Add new zed_interfaces package

* Removed "world_frame"

* removed "_m" from parameters

* Remove publish_pose_covariance parameter

* - Rename `depth_resample_factor` to `depth_downsample_factor`
- Rename `img_resample_factor` to `img_downsample_factor`

* Rename `odometry_db` to `area_memory_db_path`

* Update Changelog

* Support for Textureness Depth Threshold

* Minor fixes

* ZED2 sensors frames

* Improved warning message for missing TF transforms

* Minor fixes

* Minor fix

* Feat gray images (#532)

* Improved warning message for missing TF transforms
* Minor fixes
* Add gray images publishing
* Gray image publishing correctly working

* Camera IMU transform publisher

* Left Camera to IMU transform new topic name `left_camera_imu_transform`

* Default value for depth_confidence to 50

* Propagate `base_frame` parameter in the Xacro description

* Fix zed_no_tf.launch

* Add support for new Sensor Information info structures
Add support for new extrinsic parameters in ROS frame

* Update LICENSE

* Add separated publishing frequency for Video and Depth data
Add new publishing frequency info to diagnostic
Add new publishing frequency to dynamic parameters

* Solve conflicts

File: zed_wrapper/urdf/zed_descr.urdf.xacro (robot description, xacro)
@@ -21,4 +21,5 @@
     <xacro:arg name="camera_name"   default="zed" />
     <xacro:arg name="camera_model"  default="zed" />
+    <xacro:arg name="base_frame"    default="base_link" />
     <xacro:arg name="cam_pos_x"     default="0.0" />
     <xacro:arg name="cam_pos_y"     default="0.0" />
@@ -40,8 +41,8 @@
     </xacro:if>
 <!-- base_link -->
-    <link name="base_link" />
+    <link name="$(arg base_frame)" />
 <!-- Camera Center -->
     <joint name="$(arg camera_name)_camera_center_joint" type="fixed">
-        <parent link="base_link"/>
+        <parent link="$(arg base_frame)"/>
         <child link="$(arg camera_name)_camera_center"/>
         <origin xyz="$(arg cam_pos_x) $(arg cam_pos_y) $(arg cam_pos_z)" rpy="$(arg cam_roll) $(arg cam_pitch) $(arg cam_yaw)" />
@@ -82,3 +83,30 @@
     </joint>
     <link name="$(arg camera_name)_right_camera_optical_frame"/>
+<!-- ZED2 Sensors -->
+    <xacro:if value="${model == 'zed2'}">
+        <joint name="$(arg camera_name)_mag_joint" type="fixed">
+            <parent link="$(arg camera_name)_camera_center"/>
+            <child link="$(arg camera_name)_mag_link"/>
+            <origin xyz="0 0 0" rpy="0 0 0" />
+        </joint>
+        <link name="$(arg camera_name)_mag_link" />
+        <joint name="$(arg camera_name)_baro_joint" type="fixed">
+            <parent link="$(arg camera_name)_camera_center"/>
+            <child link="$(arg camera_name)_baro_link"/>
+            <origin xyz="0 0 0" rpy="0 0 0" />
+        </joint>
+        <link name="$(arg camera_name)_baro_link" />
+        <joint name="$(arg camera_name)_temp_left_joint" type="fixed">
+            <parent link="$(arg camera_name)_left_camera_frame"/>
+            <child link="$(arg camera_name)_temp_left_link"/>
+            <origin xyz="0 0 0" rpy="0 0 0" />
+        </joint>
+        <link name="$(arg camera_name)_temp_left_link" />
+        <joint name="$(arg camera_name)_temp_right_joint" type="fixed">
+            <parent link="$(arg camera_name)_right_camera_frame"/>
+            <child link="$(arg camera_name)_temp_right_link"/>
+            <origin xyz="0 0 0" rpy="0 0 0" />
+        </joint>
+        <link name="$(arg camera_name)_temp_right_link" />
+    </xacro:if>
 </robot>

Commit message: Moved cameras meshes STL files to zed_interfaces

File: zed_wrapper/urdf/zed_descr.urdf.xacro (robot description, xacro)
@@ -55,5 +55,5 @@
             <origin xyz="0 0 0" rpy="0 0 0"/>
             <geometry>
-                <mesh filename="package://zed_wrapper/urdf/models/${model}.stl" />
+                <mesh filename="package://zed_interfaces/meshes/${model}.stl" />
             </geometry>
             <material name="${model}_mat" />

Commit message: Create a macro that can be used to add multiple zed cameras to an existing URDF.  Make the base-link connect to the mounting hole of the camera instead of the camera's center (makes attaching the camera to a mounting point on another URDF easier).

File: zed_wrapper/urdf/zed_descr.urdf.xacro (robot description, xacro)
@@ -16,100 +16,17 @@
 -->
 <robot name="stereolabs_camera" xmlns:xacro="http://ros.org/wiki/xacro">
-<!-- Includes -->
-    <xacro:include filename="$(find zed_wrapper)/urdf/include/materials.urdf.xacro" />
-    <!-- Arguments -->
-    <xacro:arg name="camera_name"   default="zed" />
-    <xacro:arg name="camera_model"  default="zed" />
-    <xacro:arg name="base_frame"    default="base_link" />
-    <xacro:arg name="cam_pos_x"     default="0.0" />
-    <xacro:arg name="cam_pos_y"     default="0.0" />
-    <xacro:arg name="cam_pos_z"     default="0.0" />
-    <xacro:arg name="cam_roll"      default="0.0" />
-    <xacro:arg name="cam_pitch"     default="0.0" />
-    <xacro:arg name="cam_yaw"       default="0.0" />
-    <!-- Properties -->
-    <xacro:property name="M_PI"     value="3.1415926535897931" />
-    <xacro:property name="model"    value="$(arg camera_model)" />
-    <xacro:if value="${model == 'zed'}">
-        <xacro:property name="baseline" value="0.12" />
-    </xacro:if>
-    <xacro:if value="${model == 'zedm'}">
-        <xacro:property name="baseline" value="0.06" />
-    </xacro:if>
-    <xacro:if value="${model == 'zed2'}">
-        <xacro:property name="baseline" value="0.12" />
-    </xacro:if>
-    <xacro:if value="${model == 'zed2i'}">
-        <xacro:property name="baseline" value="0.12" />
-    </xacro:if>
-<!-- base_link -->
-    <link name="$(arg base_frame)" />
-<!-- Camera Center -->
-    <joint name="$(arg camera_name)_camera_center_joint" type="fixed">
-        <parent link="$(arg base_frame)"/>
-        <child link="$(arg camera_name)_camera_center"/>
-        <origin xyz="$(arg cam_pos_x) $(arg cam_pos_y) $(arg cam_pos_z)" rpy="$(arg cam_roll) $(arg cam_pitch) $(arg cam_yaw)" />
-    </joint>
-    <link name="$(arg camera_name)_camera_center">
-        <visual>
-            <origin xyz="0 0 0" rpy="0 0 0"/>
-            <geometry>
-                <mesh filename="package://zed_interfaces/meshes/${model}.stl" />
-            </geometry>
-            <material name="${model}_mat" />
-        </visual>
-    </link>
-<!-- Left Camera -->
-    <joint name="$(arg camera_name)_left_camera_joint" type="fixed">
-        <parent link="$(arg camera_name)_camera_center"/>
-        <child link="$(arg camera_name)_left_camera_frame"/>
-        <origin xyz="0 ${baseline/2} 0" rpy="0 0 0" />
-    </joint>
-    <link name="$(arg camera_name)_left_camera_frame" />
-    <joint name="$(arg camera_name)_left_camera_optical_joint" type="fixed">
-        <origin xyz="0 0 0" rpy="-${M_PI/2} 0.0 -${M_PI/2}"/>
-        <parent link="$(arg camera_name)_left_camera_frame"/>
-        <child link="$(arg camera_name)_left_camera_optical_frame"/>
-    </joint>
-    <link name="$(arg camera_name)_left_camera_optical_frame"/>
-<!-- Right Camera -->
-    <joint name="$(arg camera_name)_right_camera_joint" type="fixed">
-        <parent link="$(arg camera_name)_camera_center"/>
-        <child link="$(arg camera_name)_right_camera_frame"/>
-        <origin xyz="0 -${baseline/2} 0" rpy="0 0 0" />
-    </joint>
-    <link name="$(arg camera_name)_right_camera_frame" />
-    <joint name="$(arg camera_name)_right_camera_optical_joint" type="fixed">
-        <origin xyz="0 0 0" rpy="-${M_PI/2} 0.0 -${M_PI/2}"/>
-        <parent link="$(arg camera_name)_right_camera_frame"/>
-        <child link="$(arg camera_name)_right_camera_optical_frame"/>
-    </joint>
-    <link name="$(arg camera_name)_right_camera_optical_frame"/>
-<!-- ZED2 Sensors -->
-    <xacro:if value="${model == 'zed2'}">
-        <joint name="$(arg camera_name)_mag_joint" type="fixed">
-            <parent link="$(arg camera_name)_camera_center"/>
-            <child link="$(arg camera_name)_mag_link"/>
-            <origin xyz="0 0 0" rpy="0 0 0" />
-        </joint>
-        <link name="$(arg camera_name)_mag_link" />
-        <joint name="$(arg camera_name)_baro_joint" type="fixed">
-            <parent link="$(arg camera_name)_camera_center"/>
-            <child link="$(arg camera_name)_baro_link"/>
-            <origin xyz="0 0 0" rpy="0 0 0" />
-        </joint>
-        <link name="$(arg camera_name)_baro_link" />
-        <joint name="$(arg camera_name)_temp_left_joint" type="fixed">
-            <parent link="$(arg camera_name)_left_camera_frame"/>
-            <child link="$(arg camera_name)_temp_left_link"/>
-            <origin xyz="0 0 0" rpy="0 0 0" />
-        </joint>
-        <link name="$(arg camera_name)_temp_left_link" />
-        <joint name="$(arg camera_name)_temp_right_joint" type="fixed">
-            <parent link="$(arg camera_name)_right_camera_frame"/>
-            <child link="$(arg camera_name)_temp_right_link"/>
-            <origin xyz="0 0 0" rpy="0 0 0" />
-        </joint>
-        <link name="$(arg camera_name)_temp_right_link" />
-    </xacro:if>
+  <xacro:arg name="camera_name"   default="zed" />
+  <xacro:arg name="camera_model"  default="zed" />
+  <xacro:arg name="base_frame"    default="base_link" />
+  <xacro:arg name="cam_pos_x"     default="0.0" />
+  <xacro:arg name="cam_pos_y"     default="0.0" />
+  <xacro:arg name="cam_pos_z"     default="0.0" />
+  <xacro:arg name="cam_roll"      default="0.0" />
+  <xacro:arg name="cam_pitch"     default="0.0" />
+  <xacro:arg name="cam_yaw"       default="0.0" />
+  <xacro:include filename="$(find zed_wrapper)/urdf/zed_macro.urdf.xacro" />
+  <xacro:zed_camera name="${camera_name}" model="${camera_model}" parent="${base_frame}">
+    <origin xyz="${cam_pos_x} ${cam_pos_y} ${cam_pos_z}" rpy="${cam_roll} ${cam_pitch} ${cam_yaw}" />
+  </xacro:zed_camera>
+  <link name="${base_frame}" />
 </robot>

Commit message: Fix syntax errors in xacro file and improve URDF

File: zed_wrapper/urdf/zed_descr.urdf.xacro (robot description, xacro)
@@ -26,7 +26,7 @@
   <xacro:arg name="cam_yaw"       default="0.0" />
   <xacro:include filename="$(find zed_wrapper)/urdf/zed_macro.urdf.xacro" />
-  <xacro:zed_camera name="${camera_name}" model="${camera_model}" parent="${base_frame}">
-    <origin xyz="${cam_pos_x} ${cam_pos_y} ${cam_pos_z}" rpy="${cam_roll} ${cam_pitch} ${cam_yaw}" />
+  <xacro:zed_camera name="$(arg camera_name)" model="$(arg camera_model)" parent="$(arg base_frame)">
+    <origin xyz="$(arg cam_pos_x) $(arg cam_pos_y) $(arg cam_pos_z)" rpy="$(arg cam_roll) $(arg cam_pitch) $(arg cam_yaw)" />
   </xacro:zed_camera>
-  <link name="${base_frame}" />
+  <link name="$(arg base_frame)" />
 </robot>

Commit message: Update zed_descr.urdf.xacro

File: zed_wrapper/urdf/zed_descr.urdf.xacro (robot description, xacro)
@@ -34,13 +34,3 @@
   </xacro:zed_camera>
   <link name="$(arg base_frame)" />
-  <xacro:property name="gnss_frame" value="$(arg gnss_frame)"/>
-  <!-- Set the position of the GNSS sensor relative to base_link if used -->
-  <xacro:if value="${gnss_frame != ''}">
-    <link name="$(arg gnss_frame)" />
-    <joint name="$(arg gnss_frame)_joint" type="fixed">
-      <parent link="$(arg base_frame)"/>
-      <child link="$(arg gnss_frame)"/>
-      <origin xyz="0 0 0.5" rpy="0 0 0" />
-    </joint>
-  </xacro:if>
 </robot>
